Commit message: 오케

File: urdf/cctv.urdf (robot description, URDF)
Before this commit: robot cctv, 4 links, 3 joints
Joints:
- joint joint1: origin xyz=0 0 2.012 rpy=0 0 0 -> xyz=0 0 0.712 rpy=0 0 0

Commit message: rr

File: urdf/cctv.urdf (robot description, URDF)
Before this commit: robot cctv, 4 links, 3 joints
Joints:
- joint joint1: origin xyz=0 0 0.712 rpy=0 0 0 -> xyz=0 0 0.012 rpy=0 0 0
